File: Apple2Card/Apple2Card.kicad_pcb (KiCad board)
At the start: 2 copper layers, 160 x 78.7 mm, 77 parts, among them J1 ICSP, J2 Conn_01x25, J3 Conn_01x25, J4 Conn_01x16, J5 SERCON, J6 WIZNET 5500, SW1 SW_Push, U1 ATmega328P-P, U2 74HCT32, U3 74HCT00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

Commit message: Added interactive BOM.
Parts:
- U5: footprint Apple2Card:MicroSD_Card_TB -> Apple2Card:GCT-MEM2055-00-190-01-A
Changed lines of the file:
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@@
   )
   (paper "A4")
+  (title_block
+    (title "DAN ][ Controller")
+    (date "2023-10-03")
+    (rev "1.1.1")
+    (company "Apple ][ Forever!")
+  )
   (layers
     (0 "F.Cu" signal)
@@
     )
   )
-  (footprint "Apple2Card:MicroSD_Card_TB" (layer "F.Cu")
+  (footprint "Apple2Card:GCT-MEM2055-00-190-01-A" (layer "F.Cu")
     (at 46.52 73.91 90)
     (descr "http://www.farnell.com/datasheets/1917242.pdf")
